File: pcb/PCA9685 Replica.sch (KiCad schematic (older format))
At the start: 62 parts, among them J1 Conn_01x03, J10 Conn_01x03, J11 Conn_01x03, J12 Conn_01x03, J13 Conn_01x03, J14 Conn_01x03, J15 Conn_01x03, J16 Conn_01x03, J17 Screw_Terminal_01x02, J18 Conn_01x06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

Commit message: update project
Parts:
- J1, J10, J11, J12, J13, J14, J15, J16, J2, J3, J4, J5, J6, J7, J8, J9: Código (none) -> NRC003SAAN-RC(Digikey)
- J18: Código (none) -> NRC006SAAN-RC (Digikey)
- Q1: Código (none) -> SUD50P08-25L-E3CT-ND
- R1, R2, R23, R24, R3, R4, R5, R6, R7: Código (none) -> RC0805DK0710KL(Digikey)
- R10, R11, R12, R13, R14, R15, R16, R17, R18, R19, R20, R21, R25, R26, R8, R9: Código (none) -> RC0805DK07220L(Digikey)
- R22: Código (none) -> RC0805DK07470L(Digikey)
- U1: Código (none) -> 568-11925-6-ND(Digikey)
Other:
- note added: "1- +V\n2- GND"
- note added: "Bloque de control de servos mediante I2C\n"
- note removed: "Bloque principal con PCA9685\n"
