File: pcb/PCA9685 Replica.kicad_pcb (KiCad board)
At the start: 2 copper layers, 63 x 50 mm, 62 parts, among them J1 Conn_01x03, J10 Conn_01x03, J11 Conn_01x03, J12 Conn_01x03, J13 Conn_01x03, J14 Conn_01x03, J15 Conn_01x03, J16 Conn_01x03, J17 Screw_Terminal_01x02, J18 Conn_01x06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

Commit message: update project
Parts:
- added REF**: OSHW-Logo2_7.3x6mm_SilkScreen, Symbol:OSHW-Logo2_7.3x6mm_SilkScreen, F.Cu at (125.8, 114.0)
- moved R7 29.8 mm to (118.5, 110.5), turned to 270 degrees
- moved FID2 28.5 mm to (114.5, 119.5)
- moved Q1 12.5 mm to (135.5, 86.1)
- moved J17 8.51 mm to (127.5, 85.5)
- moved R23 6.18 mm to (118.5, 101.4)
- moved R24 6.18 mm to (118.5, 97.4)
- moved C2 4.61 mm to (131.0, 104.5)
- moved C1 4.46 mm to (139.5, 105.2)
- moved R22 3.35 mm to (118.5, 114.9)
- moved FID1 2.69 mm to (114.5, 91.0)
- moved D1 2.50 mm to (118.5, 106.0)
- moved R6 2.01 mm to (137.7, 120.2)
- moved R5 2.00 mm to (135.0, 120.2), turned to 270 degrees
- moved R4 2.00 mm to (132.2, 120.2), turned to 270 degrees
- moved R3 2.00 mm to (129.5, 120.2)
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Routing:
- net +5V: track 0.00 -> 137.8 mm
- net GND: track 0.00 -> 97.1 mm, vias 0 -> 3
- net VCC: track 0.00 -> 96.5 mm, vias 0 -> 1
- net /OE: track 0.00 -> 88.1 mm, vias 0 -> 1
- net /SCL: track 0.00 -> 50.2 mm, vias 0 -> 1
- net /SDA: track 0.00 -> 49.0 mm, vias 0 -> 1
- net /A5: track 0.00 -> 46.0 mm, vias 0 -> 2
- net /A0: track 0.00 -> 42.7 mm
- net /A1: track 0.00 -> 42.4 mm, vias 0 -> 2
- net /A2: track 0.00 -> 40.1 mm, vias 0 -> 2
- net /A3: track 0.00 -> 38.1 mm, vias 0 -> 2
- net /A4: track 0.00 -> 35.9 mm, vias 0 -> 2
- net /PWM4: track 0.00 -> 15.3 mm
- net /PWM11: track 0.00 -> 14.6 mm
- net /PWM0: track 0.00 -> 14.6 mm
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- added copper zone on B.Cu, net GND
Other:
- net class Default: clearance 0.5 -> 0.3; trace_width 0.5 -> 0.8; via_dia 1.4 -> 1.6; via_drill 0.7 -> 0.8
- net class net_PCA9685 removed
- rule trace_clearance: 0.5 -> 0.3
- board text added: "+5V"
- board text added: "+V"
- board text added: "0"
- board text added: "1"
- board text added: "10"
- board text added: "11"
- board text added: "12"
- board text added: "13"
- board text added: "14"
- board text added: "15"
- board text added: "2"
- board text added: "3"
- board text added: "4"
- board text added: "5"
- board text added: "6"
- board text added: "7"
- board text added: "8"
- board text added: "9"
- board text added: "A0"
- board text added: "A1"
- board text added: "A2"
- board text added: "A3"
- board text added: "A4"
- board text added: "A5"
- board text added: "Adafruit 16-Channel PWM/Servo Driver (Réplica)"
- board text added: "Ancho de pista: - 0,8 mm - 0,5 mm - 0,25 mm"
- board text added: "Clearance 0,3 mm"
- board text added: "Datos de referencia del fabricante: Mayer S.A"
- board text added: "Espesor de Cobre: 1oz Espesor de la tarjeta PCB: 1,6 mm Acabado Superficial: HASL"
- board text added: "GND"
- board text added: "Gerónimo Franco"
- board text added: "Grillas: - de posicionamiento: 1 mm - 0,5 mm - 0,25 mm - de ruteo: 1 mm - 0,5 mm"
- board text added: "Ind. Arg."
- board text added: "Notas para el proceso de fabricación:"
- board text added: "N° de capas: 2"
- board text added: "OE"
- board text added: "PWM"
- board text added: "Rev: 1.0"
- board text added: "SCL"
- board text added: "SDA"
- board text added: "VCC"
- board text added: "Vias: 1,6 mm / 0,8 mm"

Commit message: update pcb
Other:
- board text added: "Vias: - 1,6 mm / 0,8 mm - 1.4 mm / 0.7 mm"
- board text removed: "Vias: 1,6 mm / 0,8 mm"

Commit message: update
Other:
- board text added: "Minimo 10 mils Espesor de Cobre: 1oz Espesor de la tarjeta PCB: 1,6 mm Acabado Superficial: HASL"
- board text removed: "Espesor de Cobre: 1oz Espesor de la tarjeta PCB: 1,6 mm Acabado Superficial: HASL"
